File: FET_Driver/FET_Driver.sch (KiCad schematic (older format))
At the start: 8 parts, among them J101 Interface, J102 Out, Q101 IRF5210SPbF, U101 EL3H7(C)(TA)-G

Commit message: Fix Libraries
Parts:
- Q101: symbol FET_Driver:IRF5210SPbF -> YachtHardware:IRF5210SPbF
- U101: symbol SH-ESP32:EL3H7 -> YachtHardware:EL3H7
Changed lines of the file:
@@
 GPIO
 $Comp
-L FET_Driver:IRF5210SPbF Q101
+L YachtHardware:IRF5210SPbF Q101
 U 1 1 5FB80F51
 P 5250 3450
@@
 Flyback diode for inductive loads
 $Comp
-L SH-ESP32:EL3H7 U101
+L YachtHardware:EL3H7 U101
 U 1 1 5FCB38F6
 P 3850 3550

Commit message: Re-arrange FET Driver  PCB  for better High current tracks
Parts:
- added D502: GREEN LED, LED_SMD:LED_0603_1608Metric, symbol Device:LED
- added R502: 1k, Resistor_SMD:R_0603_1608Metric, symbol Device:R
- Q101: value IRF5210SPbF -> IRF5210STRLPBF; LCSC (none) -> C2622
- R101: LCSC (none) -> C25804
- R102: LCSC (none) -> C21190
Connections:
- wire segments 31 -> 35
Other:
- moved on the sheet: D101, J102, Q101, R101, R102, R901, U101

Commit message: Change FET VIN/OUT connector to 4 Pin to reduce stock parts
Parts:
- J102: footprint Connector_Phoenix_MC:PhoenixContact_MCV_1,5_3-G-3.81_1x03_P3.81mm_Vertical -> Connector_Phoenix_MC:PhoenixContact_MCV_1,5_4-G-3.81_1x04_P3.81mm_Vertical; symbol Connector_Generic:Conn_01x03 -> Connector_Generic:Conn_01x04
- renumbered D502 to D102, R502 to R103
Connections:
- wire segments 35 -> 36
Changed lines of the file:
@@
 $EndComp
 $Comp
-L Connector_Generic:Conn_01x03 J102
+L Connector_Generic:Conn_01x04 J102
 U 1 1 5FB9C499
 P 8000 3400
 F 0 "J102" H 8080 3442 50  0000 L CNN
 F 1 "Out" H 8080 3351 50  0000 L CNN
-F 2 "Connector_Phoenix_MC:PhoenixContact_MCV_1,5_3-G-3.81_1x03_P3.81mm_Vertical" H 8000 3400 50  0001 C CNN
+F 2 "Connector_Phoenix_MC:PhoenixContact_MCV_1,5_4-G-3.81_1x04_P3.81mm_Vertical" H 8000 3400 50  0001 C CNN
 F 3 "~" H 8000 3400 50  0001 C CNN
 	1    8000 3400
@@
 $EndComp
 $Comp
-L Device:LED D?
+L Device:LED D102
 U 1 1 5FC5F82B
 P 2950 3950
-AR Path="/5FC5F82B" Ref="D?"  Part="1"
+AR Path="/5FC5F82B" Ref="D102"  Part="1"
 AR Path="/5FC50B89/5FC5F82B" Ref="D502"  Part="1"
-F 0 "D?" V 2989 3832 50  0000 R CNN
+F 0 "D102" V 2989 3832 50  0000 R CNN
 F 1 "GREEN LED" V 2898 3832 50  0000 R CNN
 F 2 "LED_SMD:LED_0603_1608Metric" H 2950 3950 50  0001 C CNN
@@
 $EndComp
 $Comp
-L Device:R R?
+L Device:R R103
 U 1 1 5FC5F831
 P 2950 3450
-AR Path="/5FC5F831" Ref="R?"  Part="1"
+AR Path="/5FC5F831" Ref="R103"  Part="1"
 AR Path="/5FC50B89/5FC5F831" Ref="R502"  Part="1"
-F 0 "R?" H 3020 3496 50  0000 L CNN
+F 0 "R103" H 3020 3496 50  0000 L CNN
 F 1 "1k" H 3020 3405 50  0000 L CNN
 F 2 "Resistor_SMD:R_0603_1608Metric" V 2880 3450 50  0001 C CNN
@@
 Wire Wire Line
 	2950 4100 2950 4300
+Wire Wire Line
+	7800 3500 7800 3600
+Connection ~ 7800 3500
 $EndSCHEMATC
